File: electronics/StickPassV2.kicad_pcb (KiCad board)
At the start: 2 copper layers, 50 x 18.2 mm, 12 parts, among them IC1 ATTINY85-P, P1 USB_A, SW1 SW_PUSH

Commit message: Update electronic schematic and add gerber files.
Parts:
- IC1: footprint Housings_DIP:DIP-8_W7.62mm -> stickpass:DIP-8_W7.62mm
- P1: footprint Connect:USB_A -> Connect:usb_a_molex_48037-0001
- moved D1 3.50 mm to (122.0, 88.5)
- moved D2 3.50 mm to (121.9, 85.0)
- moved R4 3.50 mm to (117.6, 85.0)
- moved R3 3.25 mm to (117.6, 88.2)
- moved P1 0.70 mm to (104.8, 85.3)
Routing:
- net +5V: track 0.00 -> 30.9 mm
- net D-: track 23.5 -> 29.9 mm
- net Net-(D3-Pad1): track 11.7 -> 17.0 mm
- net D+: track 18.2 -> 19.7 mm
- net IC+: track 18.6 -> 17.9 mm
- net IC-: track 17.5 -> 18.2 mm, vias 0 -> 1
Other:
- net class Default: clearance 0.25 -> 0.3
- rule trace_clearance: 0.25 -> 0.3
- rule trace_min: 0.3 -> 0.2
- rule via_min_drill: 0.3 -> 0.2
