File: electronics/StickPassV2.sch (KiCad schematic (older format))
At the start: 12 parts, among them IC1 ATTINY85-P, P1 USB_A, SW1 SW_PUSH, SW2 SW_PUSH

Commit message: Update electronic circuit files.
Parts:
- removed R2: 10K, symbol R
- removed SW2: SW_PUSH, symbol SW_PUSH
- added D3: LED, LEDs:LED-5MM, symbol LED
- added R5: 220R, Resistors_ThroughHole:Resistor_Horizontal_RM10mm, symbol R
- C1: value 100n -> 0.1u; footprint (none) -> Resistors_ThroughHole:Resistor_Horizontal_RM7mm
- D1, D2: footprint (none) -> Resistors_ThroughHole:Resistor_Horizontal_RM7mm
- IC1: footprint DIP8 -> Housings_DIP:DIP-8_W7.62mm
- P1: footprint (none) -> Connect:USB_A
- R1: footprint (none) -> Resistors_ThroughHole:Resistor_Horizontal_RM10mm
- R2: renamed from R3; footprint (none) -> Resistors_ThroughHole:Resistor_Horizontal_RM10mm
- R3: renamed from R4; footprint (none) -> Resistors_ThroughHole:Resistor_Horizontal_RM7mm
- R4: renamed from R5; footprint (none) -> Resistors_ThroughHole:Resistor_Horizontal_RM7mm
- SW1: footprint (none) -> switch:SPST-4-PIN_6mm_thru
Connections:
- net GND: now also R5.2
- net IC-: now reaches IC1.6 (PB1(MISO/DO/AIN1/OC0B/OC1A/PCINT1)), R3.1
- net IC+: now reaches IC1.7 (PB2(SCK/USCK/SCL/T0/INT0/ADC1/PCINT2)), R4.1
- net PB1: no longer names the net of IC1.3 (PB4(XTAL2/CLKO/OC1B/ADC2/PCINT4))
- net PB1: now also D3.2 (A)
- new net: D3.1 (K), R5.1
Other:
- note removed: "Microcontroller"
- note removed: "POWER FLAGS"
- note removed: "Pushbuttons"
- note removed: "USB"
- moved on the sheet: C1, D1, D2, IC1, P1, R1, R2, R3, R4, SW1

Commit message: Update electronic schematic and add gerber files.
Parts:
- IC1: footprint Housings_DIP:DIP-8_W7.62mm -> stickpass:DIP-8_W7.62mm
- P1: footprint Connect:USB_A -> Connect:usb_a_molex_48037-0001
Changed lines of the file:
@@
 F 0 "IC1" H 5950 4100 40  0000 C CNN
 F 1 "ATTINY85-P" H 8100 3300 40  0000 C CNN
-F 2 "Housings_DIP:DIP-8_W7.62mm" H 8100 3700 35  0001 C CIN
+F 2 "stickpass:DIP-8_W7.62mm" H 8100 3700 35  0001 C CIN
 F 3 "" H 7100 3700 60  0000 C CNN
 	1    7100 3700
@@
 F 0 "P1" H 4000 2950 50  0000 C CNN
 F 1 "USB_A" H 3750 3350 50  0000 C CNN
-F 2 "Connect:USB_A" V 3750 3050 60  0001 C CNN
+F 2 "Connect:usb_a_molex_48037-0001" V 3750 3050 60  0001 C CNN
 F 3 "" V 3750 3050 60  0000 C CNN
 	1    3800 3150
